File: Aukey Fuel Gauge.kicad_pcb (KiCad board)
At the start: 2 copper layers, 30.6 x 12.4 mm, 19 parts, among them P1 DC In, SW1 Batt Test, U1 LM3914

Commit message: Initial commit
Added Solder Jumper into schematic for Mode selection. Schematic is done. PCB Layout is laid out but still needs traces run and part designed for Jumper.
Other:
- board text added: "Aukey Battery Fuel Gauge v1.1 2017 Optoisolated"
- board text removed: "Aukey Battery Fuel Gauge v1.1 2017 MATDAR"
Changed lines of the file:
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@@
-(kicad_pcb (version 20171130) (host pcbnew "(5.0.0)")
+(kicad_pcb (version 20171130) (host pcbnew "(5.0.2)-1")
   (general
     (thickness 1.6)
@@
     (pad_drill 0.762)
     (pad_to_mask_clearance 0.2)
+    (solder_mask_min_width 0.25)
     (aux_axis_origin 0 0)
     (visible_elements 7FFFFFFF)
@@
   (gr_line (start 131.4 100.9) (end 130.6 101.7) (angle 90) (layer Edge.Cuts) (width 0.15))
   (gr_line (start 161.2 101.5) (end 160.6 100.9) (angle 90) (layer Edge.Cuts) (width 0.15))
-  (gr_text "Aukey Battery\nFuel Gauge v1.1\n2017 MATDAR" (at 131.5 102.4) (layer B.SilkS)
+  (gr_text "Aukey Battery\nFuel Gauge v1.1\n2017 Optoisolated" (at 131.5 102.4) (layer B.SilkS)
     (effects (font (size 0.4 0.4) (thickness 0.1)) (justify right mirror))
   )
