File: Aukey Fuel Gauge.sch (KiCad schematic (older format))
At the start: 19 parts, among them P1 DC In, SW1 Batt Test, U1 LM3914

Commit message: Initial commit
Added Solder Jumper into schematic for Mode selection. Schematic is done. PCB Layout is laid out but still needs traces run and part designed for Jumper.
Parts:
- added JP1: Mode, symbol Jumper:SolderJumper_2_Open
- C1: symbol C_Small -> Aukey-Fuel-Gauge-rescue:C_Small
- D1, D10, D2, D3, D4, D5, D6, D7, D8, D9: symbol Led_Small -> Aukey-Fuel-Gauge-rescue:Led_Small
- P1: symbol CONN_01X02 -> Aukey-Fuel-Gauge-rescue:CONN_01X02
- R1, R2, R3, R4, R5: symbol R -> Aukey-Fuel-Gauge-rescue:R
- SW1: symbol SW_PUSH -> Aukey-Fuel-Gauge-rescue:SW_PUSH
- U1: symbol LM3914 -> Aukey-Fuel-Gauge-rescue:LM3914
Connections:
- net GND: now also JP1.1 (A)
- net at U1.11 (Mode): now also JP1.2 (B)
- no-connect marks 1 -> 0
Other:
- note added: "Open for Dot Mode\nClose for Bar Mode\n"
- note removed: "Open for\nDot Mode\n"
Changed lines of the file:
@@
-EESchema Schematic File Version 2
-LIBS:power
-LIBS:device
-LIBS:transistors
-LIBS:conn
-LIBS:linear
-LIBS:regul
-LIBS:74xx
-LIBS:cmos4000
-LIBS:adc-dac
-LIBS:memory
-LIBS:xilinx
-LIBS:microcontrollers
-LIBS:dsp
-LIBS:microchip
-LIBS:analog_switches
-LIBS:motorola
-LIBS:texas
-LIBS:intel
-LIBS:audio
-LIBS:interface
-LIBS:digital-audio
-LIBS:philips
-LIBS:display
-LIBS:cypress
-LIBS:siliconi
-LIBS:opto
-LIBS:atmel
-LIBS:contrib
-LIBS:valves
-LIBS:Aukey Parts
+EESchema Schematic File Version 4
 LIBS:Aukey Fuel Gauge-cache
-EELAYER 25 0
+EELAYER 26 0
 EELAYER END
 $Descr A4 11693 8268
@@
 $EndDescr
 $Comp
-L LM3914 U1
+L Aukey-Fuel-Gauge-rescue:LM3914 U1
 U 1 1 583BEC7A
 P 5000 3450
@@
 4.2V (8.4v)max per cell\n3.0V (6.0v)min per cell\n\n(2 cells in series) x4\n\n
 $Comp
-L R R4
+L Aukey-Fuel-Gauge-rescue:R R4
 U 1 1 583BED8E
 P 4125 3300
@@
 $EndComp
 $Comp
-L R R3
+L Aukey-Fuel-Gauge-rescue:R R3
 U 1 1 583BEDE3
 P 3600 3700
@@
 $EndComp
 $Comp
-L R R1
+L Aukey-Fuel-Gauge-rescue:R R1
 U 1 1 583BEE5F
 P 3425 3300
@@
 $EndComp
 $Comp
-L R R2
+L Aukey-Fuel-Gauge-rescue:R R2
 U 1 1 583BEE92
 P 3425 3700
@@
 $EndComp
 Wire Wire Line
-	4550 3300 4275 3300
-Wire Wire Line
-	3750 3300 3975 3300
+	4550 3300 4350 3300
+Wire Wire Line
+	3750 3300 3850 3300
 Wire Wire Line
 	3925 3200 4550 3200
@@
 	3425 3500 4550 3500
 Wire Wire Line
-	3425 3450 3425 3550
+	3425 3450 3425 3500
 Connection ~ 3425 3500
 $Comp
-L +BATT #PWR01
+L Aukey-Fuel-Gauge-rescue:+BATT #PWR01
 U 1 1 583BF31F
 P 2825 2775
@@
 $EndComp
 Wire Wire Line
-	3425 2775 3425 3150
-$Comp
-L C_Small C1
+	3425 2775 3425 2825
+$Comp
+L Aukey-Fuel-Gauge-rescue:C_Small C1
 U 1 1 583BF4B2
 P 4150 2850
@@
 $EndComp
 $Comp
-L GND #PWR02
+L Aukey-Fuel-Gauge-rescue:GND #PWR02
 U 1 1 583BF6CE
 P 4325 2975
@@
 	4450 3050 4450 2975
 Wire Wire Line
-	4450 2975 4150 2975
+	4450 2975 4325 2975
 Connection ~ 4325 2975
 Wire Wire Line
 	4150 2975 4150 2950
 Wire Wire Line
-	4000 2750 4550 2750
+	4000 2750 4150 2750
 Wire Wire Line
 	4550 2750 4550 2950
@@
 	3600 3875 3425 3875
 Wire Wire Line
-	3425 3850 3425 3950
-$Comp
-L GND #PWR03
+	3425 3850 3425 3875
+$Comp
+L Aukey-Fuel-Gauge-rescue:GND #PWR03
 U 1 1 583BF8E1
 P 3425 3950
@@
 Connection ~ 4350 3300
 $Comp
-L Led_Small D1
+L Aukey-Fuel-Gauge-rescue:Led_Small D1
 U 1 1 583BFB5B
 P 5700 2950
@@
 $EndComp
 $Comp
-L Led_Small D2
+L Aukey-Fuel-Gauge-rescue:Led_Small D2
 U 1 1 583BFDD7
 P 5700 3050
@@
 $EndComp
 $Comp
-L Led_Small D3
+L Aukey-Fuel-Gauge-rescue:Led_Small D3
 U 1 1 583BFE0F
 P 5700 3150
@@
 $EndComp
 $Comp
-L Led_Small D4
+L Aukey-Fuel-Gauge-rescue:Led_Small D4
 U 1 1 583BFE3E
 P 5700 3250
@@
 $EndComp
 $Comp
-L Led_Small D5
+L Aukey-Fuel-Gauge-rescue:Led_Small D5
 U 1 1 583BFEC8
 P 5700 3350
@@
 $EndComp
 $Comp
-L Led_Small D6
+L Aukey-Fuel-Gauge-rescue:Led_Small D6
 U 1 1 583BFF05
 P 5700 3450
@@
 $EndComp
 $Comp
-L Led_Small D7
+L Aukey-Fuel-Gauge-rescue:Led_Small D7
 U 1 1 583BFF3D
 P 5700 3550
@@
 $EndComp
 $Comp
-L Led_Small D8
+L Aukey-Fuel-Gauge-rescue:Led_Small D8
 U 1 1 583BFF80
 P 5700 3650
@@
 $EndComp
 $Comp
-L Led_Small D9
+L Aukey-Fuel-Gauge-rescue:Led_Small D9
 U 1 1 583C002E
 P 5700 3750
@@
 $EndComp
 $Comp
-L Led_Small D10
+L Aukey-Fuel-Gauge-rescue:Led_Small D10
 U 1 1 583C006F
 P 5700 3850
@@
 	5800 3850 5875 3850
 Wire Wire Line
-	5875 3850 5875 2700
+	5875 3850 5875 3750
 Wire Wire Line
 	5875 2700 3950 2700
@@
 	5800 3750 5875 3750
 Connection ~ 5875 3750
-Text Notes 4300 4075 0    60   ~ 0
-Open for\nDot Mode\n
-NoConn ~ 4550 3850
-$Comp
-L SW_PUSH SW1
+Text Notes 3875 4400 0    60   ~ 0
+Open for Dot Mode\nClose for Bar Mode\n
+$Comp
+L Aukey-Fuel-Gauge-rescue:SW_PUSH SW1
 U 1 1 583C0FF7
 P 3125 2775
@@
 Capacity LEDs\n
 $Comp
-L CONN_01X02 P1
+L Aukey-Fuel-Gauge-rescue:CONN_01X02 P1
 U 1 1 583C3108
 P 2925 3575
@@
 $EndComp
 $Comp
-L +BATT #PWR04
+L Aukey-Fuel-Gauge-rescue:+BATT #PWR04
 U 1 1 583C321C
 P 2875 3375
@@
 $EndComp
 $Comp
-L GND #PWR05
+L Aukey-Fuel-Gauge-rescue:GND #PWR05
 U 1 1 583C325D
 P 3225 3400
@@
 	2675 4425 6300 4425
 $Comp
-L R R5
+L Aukey-Fuel-Gauge-rescue:R R5
 U 1 1 5844032A
 P 3600 3300
@@
 Wire Wire Line
 	3600 3100 3600 3150
+Wire Wire Line
+	3425 3500 3425 3550
+Wire Wire Line
+	4325 2975 4150 2975
+Wire Wire Line
+	3425 2975 3425 3150
+Wire Wire Line
+	4150 2750 4550 2750
+Wire Wire Line
+	3425 3875 3425 3950
+Wire Wire Line
+	4350 3300 4275 3300
+Wire Wire Line
+	3425 2825 3425 2975
+Wire Wire Line
+	5875 2950 5875 2700
+Wire Wire Line
+	5875 3050 5875 2950
+Wire Wire Line
+	5875 3150 5875 3050
+Wire Wire Line
+	5875 3250 5875 3150
+Wire Wire Line
+	5875 3350 5875 3250
+Wire Wire Line
+	5875 3450 5875 3350
+Wire Wire Line
+	5875 3550 5875 3450
+Wire Wire Line
+	5875 3650 5875 3550
+Wire Wire Line
+	5875 3750 5875 3650
+Wire Wire Line
+	3850 3300 3925 3300
+Wire Wire Line
+	3925 3300 3975 3300
+$Comp
+L Jumper:SolderJumper_2_Open JP1
+U 1 1 5CBAC11B
+P 4400 3850
+F 0 "JP1" H 4525 3900 50  0000 C CNN
+F 1 "Mode" H 4250 3900 50  0000 C CNN
+F 2 "" H 4400 3850 50  0001 C CNN
+F 3 "~" H 4400 3850 50  0001 C CNN
+	1    4400 3850
+	1    0    0    -1
+$EndComp
+$Comp
+L Aukey-Fuel-Gauge-rescue:GND #PWR06
+U 1 1 5CBAC3AA
+P 4175 3975
+F 0 "#PWR06" H 4175 3725 50  0001 C CNN
+F 1 "GND" H 4175 3825 50  0000 C CNN
+F 2 "" H 4175 3975 50  0000 C CNN
+F 3 "" H 4175 3975 50  0000 C CNN
+	1    4175 3975
+	1    0    0    -1
+$EndComp
+Wire Wire Line
+	4250 3850 4175 3850
+Wire Wire Line
+	4175 3850 4175 3975
 $EndSCHEMATC
